File: eagle_project/Digit control.brd (EAGLE design)
At the start: 80 x 68.2 mm, 29 parts, among them IC4 74HC595, IC6 40109, IC7 40109

Commit message: Added latest schema
Parts:
- added LED8: PAD-0400, ~~dpads:0400
- added R1: 100, ~~rcl:0309/15
- GND-OUT: value PAD-0500 -> PAD-0820; device ~~dpads:0500 -> ~~dpads:0820
- moved R9 2.54 mm to (25.4, 8.89)
- moved LED2 2.54 mm to (38.1, 8.89)
- moved IC7 1.27 mm to (61.0, 22.9)
Connections:
- new net LED8: IC7.13, R1.1
- new net N$14: LED8.P$1, R1.2
Routing:
- net LED8: track 0.00 -> 6.35 mm
- net VCC: track 237.5 -> 242.6 mm
- net N$14: track 0.00 -> 3.81 mm
- net LED2: track 7.62 -> 10.2 mm
- net +12V: track 127.0 -> 128.3 mm
- net LED_INPUT8: track 58.4 -> 59.7 mm
- net LED7: track 8.89 -> 10.2 mm
- net LED6: track 21.6 -> 20.3 mm
- net LED5: track 15.2 -> 14.0 mm
- net LED_INPUT6: track 50.8 -> 49.5 mm
- net LED_INPUT5: track 45.7 -> 44.5 mm
- net LED_INPUT7: track 66.0 -> 64.8 mm
Other:
- board text added: "2022-01-19"
- board text added: "Darius Kasiulevicius"
- board text removed: "2015-02-18"
- board text removed: "v2.1 DKasiulevicius"
