File: eagle_project/Digit control.sch (EAGLE design)
At the start: 29 parts, among them IC4 74HC595, IC6 40109, IC7 40109

Commit message: Added latest schema
Parts:
- added LED8: PAD-0400, ~~dpads:PAD-0400
- added R1: 100, ~~rcl:R-EU_0309/15
- GND-OUT: value PAD-0500 -> PAD-0820; device ~~dpads:PAD-0500 -> ~~dpads:PAD-0820
Connections:
- new net LED8: IC7D.OUT, R1.1
- new net N$14: LED8.P, R1.2
