File: eagle_project/Main board.brd (EAGLE design)
At the start: 92.7 x 78.4 mm, 43 parts, among them IC1 MEGA8-P, Q1 4MHz, Q2 32.768kHz, T1 2N2222, T2 2N2222

Commit message: Added latest schema
Parts:
- removed SV4: 4, con-amp-mt:S02P
- added LED1, LED2, LED3: (no value), led:LED5MM
- added PD5: 4, con-amp-mt:S02P
- added R10, R8, R9: 47k, ~~rcl:0309/15
- C2: device ~~rcl:C025-050X050 -> ~~rcl:C102-054X133
- G2: value 3V -> CR2032; device battery:BEL/P -> cr2032:CR2032-20MM
- R1: value 100k -> 30k-60k
- T2: value 2N2222 -> BC337; device transistor:TO18 -> transistor:TO92
- moved BUZ1 18.2 mm to (76.2, 29.2), turned to 270 degrees
- moved R4 14.5 mm to (76.2, 14.0), turned to 0 degrees
- moved 12V-OUT 14.0 mm to (5.08, 36.8)
- moved T1 12.6 mm to (71.8, 19.7)
- moved C1 12.0 mm to (26.7, 31.8)
- moved R5 11.6 mm to (54.6, 18.4), turned to 0 degrees
- moved SV5 8.98 mm to (5.08, 21.6)
- moved 15V 8.35 mm to (5.08, 29.8)
- moved T2 8.35 mm to (82.5, 19.7), turned to 180 degrees
- moved GND-OUT 7.18 mm to (5.08, 45.7)
- moved C10 6.35 mm to (22.9, 22.9), turned to 270 degrees
- moved BUZ2 6.35 mm to (83.8, 29.2), turned to 270 degrees
- moved G2 5.24 mm to (16.5, 64.8), turned to 270 degrees
- moved C2 5.08 mm to (74.9, 39.4)
- moved L1 4.96 mm to (33.7, 22.9), turned to 180 degrees
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- renumbered SV1 to PD2, SV2 to PD3, SV3 to PD4
Connections:
- net INPUT1 renamed PD2
- net INPUT2 renamed PD3
- net INPUT3 renamed PD4
- removed net INPUT4: IC1.11, SV4.1
- new net N$4: IC1.24, R10.1
- new net N$5: IC1.25, R9.1
- new net N$6: IC1.26, R8.1
- new net N$7: LED1.A, R10.2
- new net N$8: LED2.A, R9.2
- new net N$9: LED3.A, R8.2
- new net PD5: IC1.11, PD5.1
- net GND: now also LED1.K, LED2.K, LED3.K, PD5.2; no longer SV4.2
Routing:
- net +12V: track 182.5 -> 0.00 mm
- net VCC: track 161.5 -> 137.9 mm
- net INPUT4: track 21.6 -> 0.00 mm
- net PD5: track 0.00 -> 20.3 mm
- net N$36: track 15.3 -> 8.28 mm
- net VBAT: track 52.8 -> 45.8 mm
- net N$63: track 40.3 -> 46.1 mm
- net N$33: track 19.1 -> 24.8 mm
- net N$39: track 16.5 -> 12.1 mm
- net N$40: track 8.89 -> 12.7 mm
- net N$34: track 38.1 -> 35.6 mm
- net N$64: track 35.0 -> 32.5 mm
- net N$37: track 14.0 -> 12.5 mm
- net N$14: track 3.81 -> 5.08 mm
- net N$2: track 6.37 -> 7.00 mm
Other:
- board text added: "2022-01-19"
- board text added: "Darius Kasiulevicius"
- board text added: "OS clock V2.02"
- board text removed: "2015-02-18"
- board text removed: "DKasiulevicius"
- board text removed: "OS clock V2.0"
