File: eagle_project/Main board.sch (EAGLE design)
At the start: 43 parts, among them IC1 MEGA8-P, Q1 4MHz, Q2 32.768kHz, T1 2N2222, T2 2N2222

Commit message: Added latest schema
Parts:
- added LED1, LED2, LED3: (no value), led:LED5MM
- added R10, R8, R9: 47k, ~~rcl:R-EU_0309/15
- C2: device ~~rcl:C-EU025-050X050 -> ~~rcl:C-EU102-054X133
- G2: value 3V -> CR2032; device battery:SL-340/P -> cr2032:CR2032
- R1: value 100k -> 30k-60k
- T2: value 2N2222 -> BC337; device transistor:2N2222 -> transistor:BC337
- renumbered SV1 to PD2, SV2 to PD3, SV3 to PD4, SV4 to PD5
Connections:
- net INPUT1 renamed PD2
- net INPUT2 renamed PD3
- net INPUT3 renamed PD4
- net INPUT4 renamed PD5
- new net N$4: IC1.PC1(ADC1), R10.1
- new net N$5: IC1.PC2(ADC2), R9.1
- new net N$6: IC1.PC3(ADC3), R8.1
- new net N$7: LED1.A, R10.2
- new net N$8: LED2.A, R9.2
- new net N$9: LED3.A, R8.2
- net GND: now also LED1.C, LED2.C, LED3.C
Other:
- moved on the sheet: R15, R16
